Commit message: feat: adding altimeter to medusa vehicles

File: medusa_vehicles/mblack_vehicle/urdf/sensors.xacro (robot description, xacro)
@@ -28,4 +28,8 @@
     <origin xyz="0 0 0" rpy="0 0 0"/>
   </xacro:default_imu_macro>
+  <!-- Altimeter sensor -->
+  <xacro:medusa_altimeter namespace="${namespace}" parent_link="$(arg namespace)/base_link" suffix="">
+    <origin xyz="-0.3 0 -0.265" rpy="0 ${0.5*pi} 0"/>
+  </xacro:medusa_altimeter>
   <!-- RPT  -->
   <!--<xacro:default_rpt namespace="${namespace}" parent_link="${namespace}/base_link">-->

File: medusa_vehicles/mvector_vehicle/urdf/sensors.xacro (robot description, xacro)
@@ -28,4 +28,8 @@
     <origin xyz="0 0 0" rpy="0 0 0"/>
   </xacro:default_imu_macro>
+  <!-- Altimeter sensor -->
+  <xacro:medusa_altimeter namespace="${namespace}" parent_link="$(arg namespace)/base_link" suffix="">
+    <origin xyz="-0.3 0 -0.265" rpy="0 ${0.5*pi} 0"/>
+  </xacro:medusa_altimeter>
   <!-- Multibeam  -->
   <!--xacro:forward_multibeam_p900
