Commit message: feat: new hydrodynamic parameters for bluerov.

File: medusa_vehicles/bluerov_heavy/urdf/base.xacro (robot description, xacro)
@@ -12,9 +12,11 @@
       Vehicle's parameters (remember to enter the model parameters below)
     -->
-  <xacro:property name="mass" value="11.2"/>
+  <xacro:property name="mass" value="11.5"/>
   <!-- Vehicle's bounding box: width, length, height -->
   <xacro:property name="x_size" value="0.448"/>
-  <xacro:property name="y_size" value="0.2384"/>
-  <xacro:property name="z_size" value="0.28066"/>
+  <!--xacro:property name="y_size" value="0.2384"/-->
+  <xacro:property name="y_size" value="0.4571"/>
+  <!--xacro:property name="z_size" value="0.28066"/-->
+  <xacro:property name="z_size" value="0.2539"/>
   <!-- Volume -->
   <xacro:property name="volume" value="0.011054"/>
@@ -44,7 +46,11 @@
                 <origin xyz="${cog}" rpy="0 0 0"/>
                 <inertia
+                 ixx="0.21" ixy="0.0"  ixz="0.0"
+                 iyx="0.0"  iyy="0.245" iyz="0.0"
+                 izx="0.0"  izy="0.0"  izz="0.245" />
+                <!--inertia
                  ixx="${0.2 * mass * y_size * y_size + 0.2 * mass * z_size * z_size}" ixy="0.0" ixz="0.0"
                  iyy="${0.2 * mass * x_size * x_size + 0.2 * mass * z_size * z_size}" iyz="0.0"
-                 izz="${0.2 * mass * x_size * x_size + 0.2 * mass * y_size * y_size}" />
+                 izz="${0.2 * mass * x_size * x_size + 0.2 * mass * y_size * y_size}" /-->
             </inertial>
             <visual>

File: medusa_vehicles/bluerov_heavy/urdf/gazebo.xacro (robot description, xacro)
@@ -3,4 +3,5 @@
     <!-- Center of buoyancy -->
     <xacro:property name="bluerov_cob" value="0 0 0.3872"/>
+    <!--xacro:property name="bluerov_cob" value="0 0 0.3872"/-->
     <!-- Vehicle's actual volume (Gazebo cannot compute the volume out of the mesh) -->
     <xacro:property name="bluerov_volume" value="${volume}"/>
@@ -22,4 +23,12 @@
           <!-- Added mass: see p.28 in Berg2012 -->
           <added_mass>
+            5.5     0      0      0    0     0
+            0       12.7   0      0    0     0
+            0       0      14.57  0    0     0
+            0       0      0      0.12 0     0
+            0       0      0      0    0.12  0
+            0       0      0      0    0     0.12
+          </added_mass>
+          <!--added_mass>
             1.7182  0  0     0 0      0
             0       0  0     0 0      0
@@ -28,9 +37,9 @@
             0       0  0     0 1.2481 0
             0       0  0     0 0      0.4006
-          </added_mass>
+          </added_mass-->
           <!-- Linear damping: see p.31 in Berg2012 -->
-          <linear_damping>-11.7391 -20 -31.8678 -25 -44.9085 -5</linear_damping>
+          <linear_damping>-4.03 -6.22 -5.18 -0.07 -0.07 -3</linear_damping>
           <!-- Non-linear damping: see p.30 in Berg2012 -->
-          <quadratic_damping>0 0 0 0 0 0</quadratic_damping>
+          <quadratic_damping>-18.18 -21.66 -36.99 -1.55 -1.55 -1.55</quadratic_damping>
         </hydrodynamic_model>
       </link>

Commit message: fix: fixed some model parameters of bluerov to fit real vehicle.

File: medusa_vehicles/bluerov_heavy/urdf/base.xacro (robot description, xacro)
@@ -16,5 +16,5 @@
   <xacro:property name="x_size" value="0.448"/>
   <!--xacro:property name="y_size" value="0.2384"/-->
-  <xacro:property name="y_size" value="0.4571"/>
+  <xacro:property name="y_size" value="0.338"/>
   <!--xacro:property name="z_size" value="0.28066"/-->
   <xacro:property name="z_size" value="0.2539"/>
@@ -52,5 +52,5 @@
                  ixx="${0.2 * mass * y_size * y_size + 0.2 * mass * z_size * z_size}" ixy="0.0" ixz="0.0"
                  iyy="${0.2 * mass * x_size * x_size + 0.2 * mass * z_size * z_size}" iyz="0.0"
-                 izz="${0.2 * mass * x_size * x_size + 0.2 * mass * y_size * y_size}" /-->
+                 izz="${0.2 * mass * x_size * x_size + 0.2 * mass * y_size * y_size}"/-->
             </inertial>
             <visual>

File: medusa_vehicles/bluerov_heavy/urdf/gazebo.xacro (robot description, xacro)
@@ -2,5 +2,5 @@
 <robot xmlns:xacro="http://www.ros.org/wiki/xacro">
     <!-- Center of buoyancy -->
-    <xacro:property name="bluerov_cob" value="0 0 0.3872"/>
+    <xacro:property name="bluerov_cob" value="0 0 0.0420"/>
     <!--xacro:property name="bluerov_cob" value="0 0 0.3872"/-->
     <!-- Vehicle's actual volume (Gazebo cannot compute the volume out of the mesh) -->
@@ -23,10 +23,10 @@
           <!-- Added mass: see p.28 in Berg2012 -->
           <added_mass>
-            5.5     0      0      0    0     0
-            0       12.7   0      0    0     0
-            0       0      14.57  0    0     0
-            0       0      0      0.12 0     0
-            0       0      0      0    0.12  0
-            0       0      0      0    0     0.12
+            27.08     0      0      0    0     0
+            0       25.952   0      0    0     0
+            0       0      29.9081  0    0     0
+            0       0      0      1  0    0
+            0       0      0      0    1  0
+            0       0      0      0    0   1
           </added_mass>
           <!--added_mass>
@@ -39,7 +39,8 @@
           </added_mass-->
           <!-- Linear damping: see p.31 in Berg2012 -->
-          <linear_damping>-4.03 -6.22 -5.18 -0.07 -0.07 -3</linear_damping>
+          <linear_damping>-0.1213 -1.1732 -1.1130 -0.5 -0.5 -0.5</linear_damping>
           <!-- Non-linear damping: see p.30 in Berg2012 -->
-          <quadratic_damping>-18.18 -21.66 -36.99 -1.55 -1.55 -1.55</quadratic_damping>
+          <!--quadratic_damping>-18.18 -21.66 -36.99 -5.55 -5.55 -5.55</quadratic_damping-->
+          <quadratic_damping>-23.9000 -46.2700 -50.2780 -1 -1 -1</quadratic_damping>
         </hydrodynamic_model>
       </link>
